Commit message: Switch default model to cart pole

File: public/urdf/cart_pole/cart_pole.urdf (robot description, URDF)
Before this commit: robot physics, 3 links, 2 joints
Links:
- link slideBar: geometry visual box size=10 0.05 0.05

Commit message: Add compass gait animation

File: public/urdf/cart_pole/cart_pole.urdf (robot description, URDF)
Before this commit: robot physics, 3 links, 2 joints
Links:
- link pole: mass 0.2 -> 1
- link slideBar: geometry visual box size=30 0.05 0.05
Joints:
- joint cart_to_pole: limit lower=-15 upper=15 effort=1000.0 velocity=5 -> lower=-50 upper=50 effort=1000.0 velocity=5
- joint slider_to_cart: limit lower=-15 upper=15 effort=1000.0 velocity=5 -> lower=-50 upper=50 effort=1000.0 velocity=5

File: public/urdf/simple/simple.urdf (robot description, URDF)
Before this commit: robot compass_gait, 9 links, 8 joints
Joints:
- joint floating_base_x: limit lower=-1.57 upper=1.57 effort=100 velocity=100 -> lower=-15 upper=15 effort=100 velocity=100
- joint floating_base_z: limit lower=-1.57 upper=1.57 effort=100 velocity=100 -> lower=-15 upper=15 effort=100 velocity=100
- joint ground_rotation: limit lower=-1.57 upper=1.57 effort=100 velocity=100 -> lower=-15 upper=15 effort=100 velocity=100
- joint hip_joint: limit lower=-1.57 upper=1.57 effort=100 velocity=100 -> lower=-15 upper=15 effort=100 velocity=100
- joint left_foot_fixed: limit lower=-1.57 upper=1.57 effort=100 velocity=100 -> lower=-15 upper=15 effort=100 velocity=100
- joint left_hip_pitch: limit lower=-1.57 upper=1.57 effort=100 velocity=100 -> lower=-15 upper=15 effort=100 velocity=100
- joint right_foot_fixed: limit lower=-1.57 upper=1.57 effort=100 velocity=100 -> lower=-15 upper=15 effort=100 velocity=100
- joint right_hip_pitch: limit lower=-1.57 upper=1.57 effort=100 velocity=100 -> lower=-15 upper=15 effort=100 velocity=100
